File: esp32_pcb/esp32_doorbot.sch (KiCad schematic (older format))
At the start: 20 parts, among them J1 Conn_01x07_Male, J2 Conn_01x02_Female, J3 Barrel_Jack, J4 WROOM32_1, J5 WROOM32_2, Q1 2N7002E, U1 L7805

Commit message: Correct mosfet pinout (for real this time)
Parts:
- removed J1: Conn_01x07_Male, Pin_Headers:Pin_Header_Straight_1x07, symbol Connector:Conn_01x07_Male
- removed J2: Conn_01x02_Female, Terminal_Blocks:TerminalBlock_Pheonix_MKDS1.5-2pol, symbol Connector:Conn_01x02_Female
- added J1: DB9_Male, Connect:DB9FD, symbol Connector:DB9_Male
- J3: footprint Terminal_Blocks:TerminalBlock_Pheonix_MKDS1.5-2pol -> Connect:BARREL_JACK; Digikey # ED2561-ND -> CP-037A-ND
- Q1: value 2N7002E -> ZVN4206GVTA; symbol Transistor_FET:2N7002E -> Transistor_FET:IRFS4227
Connections:
- net 12V: now also J1.1, J1.9
- net 5V: now also J1.2
- net GND: now also Q1.3 (S), J1.5, J1.6; no longer Q1.2 (S)
- net LATCH_OUT: now also Q1.2 (D), J1.7; no longer Q1.3 (D)
- net READER_BUZZ: now also J1.8
- net WIEGAND_IN1: now also J1.3
- net WIEGAND_IN2: now also J1.4
- net 24_32_SWITCH: no longer names the net of J4.4 (Pin_4)
- net READER_LED: no longer names the net of J4.5 (Pin_5)
- no-connect marks 21 -> 23
Changed lines of the file:
@@
 $EndDescr
 $Comp
-L Transistor_FET:2N7002E Q1
+L Transistor_FET:IRFS4227 Q1
 U 1 1 603A6F1F
 P 1450 5650
 F 0 "Q1" H 1654 5696 50  0000 L CNN
-F 1 "2N7002E" H 1654 5605 50  0000 L CNN
+F 1 "ZVN4206GVTA" H 1654 5605 50  0000 L CNN
 F 2 "TO_SOT_Packages_SMD:SOT-223" H 1650 5575 50  0001 L CIN
-F 3 "http://www.diodes.com/assets/Datasheets/ds30376.pdf" H 1450 5650 50  0001 L CNN
+F 3 "https://www.diodes.com/assets/Datasheets/ZVN4206GV.pdf" H 1450 5650 50  0001 L CNN
 F 4 "ZVN4206GVTR-ND" H 1450 5650 50  0001 C CNN "Digikey #"
 	1    1450 5650
@@
 Wire Wire Line
 	1100 5650 1200 5650
-$Comp
-L Connector:Conn_01x02_Female J2
-U 1 1 60482C20
-P 1850 3700
-F 0 "J2" H 1878 3676 50  0000 L CNN
-F 1 "Conn_01x02_Female" H 1878 3585 50  0000 L CNN
-F 2 "Terminal_Blocks:TerminalBlock_Pheonix_MKDS1.5-2pol" H 1850 3700 50  0001 C CNN
-F 3 "~" H 1850 3700 50  0001 C CNN
-F 4 "ED2561-ND" H 1850 3700 50  0001 C CNN "Digikey #"
-	1    1850 3700
-	1    0    0    -1
-$EndComp
-Text GLabel 1500 3800 0    50   Input ~ 0
+Text GLabel 3650 1050 0    50   Input ~ 0
 LATCH_IN
-Text GLabel 1500 3700 0    50   Input ~ 0
+Text GLabel 3650 1450 0    50   Input ~ 0
 LATCH_OUT
-Wire Wire Line
-	1500 3700 1650 3700
-Wire Wire Line
-	1650 3800 1500 3800
 Text GLabel 7800 3300 0    50   Input ~ 0
 DOOR
@@
 Text GLabel 4400 2950 0    50   Input ~ 0
 12V
-Text GLabel 5800 2950 2    50   Input ~ 0
-5V
 Wire Wire Line
 	4550 2950 4400 2950
@@
 Text GLabel 5050 5750 1    50   Input ~ 0
 WIEGAND_IN2
-Text GLabel 7750 2500 0    50   Input ~ 0
-READER_LED
 Text GLabel 7750 2600 0    50   Input ~ 0
 READER_BUZZ
-Text GLabel 3550 1250 0    50   Input ~ 0
+Text GLabel 3650 1750 0    50   Input ~ 0
 12V
-Text GLabel 3550 1450 0    50   Input ~ 0
+Text GLabel 3650 1350 0    50   Input ~ 0
 WIEGAND_IN1
-Text GLabel 3550 1550 0    50   Input ~ 0
+Text GLabel 3650 1150 0    50   Input ~ 0
 WIEGAND_IN2
-Text GLabel 3550 1750 0    50   Input ~ 0
-READER_LED
-Text GLabel 3550 1650 0    50   Input ~ 0
+Text GLabel 3650 1250 0    50   Input ~ 0
 READER_BUZZ
 $Comp
 L power:GND #PWR0109
 U 1 1 60644B08
-P 2800 1350
-F 0 "#PWR0109" H 2800 1100 50  0001 C CNN
-F 1 "GND" H 2805 1177 50  0000 C CNN
-F 2 "" H 2800 1350 50  0001 C CNN
-F 3 "" H 2800 1350 50  0001 C CNN
-	1    2800 1350
-	1    0    0    -1
-$EndComp
-Wire Wire Line
-	3550 1250 3750 1250
-Wire Wire Line
-	3550 1450 3750 1450
-Wire Wire Line
-	3750 1550 3550 1550
-Wire Wire Line
-	3550 1650 3750 1650
+P 3000 1650
+F 0 "#PWR0109" H 3000 1400 50  0001 C CNN
+F 1 "GND" H 3005 1477 50  0000 C CNN
+F 2 "" H 3000 1650 50  0001 C CNN
+F 3 "" H 3000 1650 50  0001 C CNN
+	1    3000 1650
+	1    0    0    -1
+$EndComp
 Text GLabel 1200 950  1    50   Input ~ 0
 12V
@@
 Wire Wire Line
 	1200 1100 1200 950
-Wire Wire Line
-	2800 1350 3750 1350
-$Comp
-L Connector:Conn_01x07_Male J1
-U 1 1 608355C5
-P 3950 1550
-F 0 "J1" V 3785 1528 50  0000 C CNN
-F 1 "Conn_01x07_Male" V 3876 1528 50  0000 C CNN
-F 2 "Pin_Headers:Pin_Header_Straight_1x07" H 3950 1550 50  0001 C CNN
-F 3 "~" H 3950 1550 50  0001 C CNN
-	1    3950 1550
-	-1   0    0    1
-$EndComp
-Wire Wire Line
-	3550 1750 3750 1750
-Text GLabel 3550 1850 0    50   Input ~ 0
-24_32_SWITCH
-Wire Wire Line
-	3550 1850 3750 1850
 $Comp
 L Connector:Barrel_Jack J3
@@
 F 0 "J3" H 5807 1775 50  0000 C CNN
 F 1 "Barrel_Jack" H 5807 1684 50  0000 C CNN
-F 2 "Terminal_Blocks:TerminalBlock_Pheonix_MKDS1.5-2pol" H 5800 1410 50  0001 C CNN
-F 3 "~" H 5800 1410 50  0001 C CNN
-F 4 "ED2561-ND" H 5750 1450 50  0001 C CNN "Digikey #"
+F 2 "Connect:BARREL_JACK" H 5800 1410 50  0001 C CNN
+F 3 "https://www.cuidevices.com/product/resource/digikeypdf/pj-037a.pdf" H 5800 1410 50  0001 C CNN
+F 4 "CP-037A-ND" H 5750 1450 50  0001 C CNN "Digikey #"
 	1    5750 1450
 	1    0    0    -1
@@
 Wire Wire Line
 	8900 2100 9050 2100
-Text GLabel 7750 2400 0    50   Input ~ 0
-24_32_SWITCH
 NoConn ~ 7950 3000
 NoConn ~ 7950 2900
@@
 NoConn ~ 7950 3100
 NoConn ~ 7950 3200
-Wire Wire Line
-	7750 2400 7950 2400
-Wire Wire Line
-	7750 2500 7950 2500
 Wire Wire Line
 	7750 2600 7950 2600
@@
 	1    0    0    -1
 $EndComp
+$Comp
+L Connector:DB9_Male J1
+U 1 1 61046136
+P 4050 1350
+F 0 "J1" H 4230 1396 50  0000 L CNN
+F 1 "DB9_Male" H 4230 1305 50  0000 L CNN
+F 2 "Connect:DB9FD" H 4050 1350 50  0001 C CNN
+F 3 "http://www.assmann-wsw.com/uploads/datasheets/ASS_4888_CO.pdf" H 4050 1350 50  0001 C CNN
+F 4 "AE10970-ND" H 4050 1350 50  0001 C CNN "Digikey #"
+	1    4050 1350
+	1    0    0    -1
+$EndComp
+Text GLabel 5800 2950 2    50   Input ~ 0
+5V
+Text GLabel 3650 1550 0    50   Input ~ 0
+5V
+$Comp
+L power:GND #PWR0112
+U 1 1 6104AFD6
+P 3000 950
+F 0 "#PWR0112" H 3000 700 50  0001 C CNN
+F 1 "GND" H 3005 777 50  0000 C CNN
+F 2 "" H 3000 950 50  0001 C CNN
+F 3 "" H 3000 950 50  0001 C CNN
+	1    3000 950
+	1    0    0    -1
+$EndComp
+Wire Wire Line
+	3750 950  3000 950
+Wire Wire Line
+	3650 1050 3750 1050
+Wire Wire Line
+	3750 1150 3650 1150
+Wire Wire Line
+	3650 1250 3750 1250
+Wire Wire Line
+	3750 1350 3650 1350
+Wire Wire Line
+	3650 1450 3750 1450
+Wire Wire Line
+	3750 1550 3650 1550
+Wire Wire Line
+	3000 1650 3750 1650
+Wire Wire Line
+	3750 1750 3650 1750
+NoConn ~ 7950 2400
+NoConn ~ 7950 2500
 $EndSCHEMATC

Commit message: Revert "Correct mosfet pinout (for real this time)"
This reverts commit 8fe08cf28d7a1d30f1efb70a8aeb7666ade41443.
Parts:
- removed J1: DB9_Male, Connect:DB9FD, symbol Connector:DB9_Male
- added J1: Conn_01x07_Male, Pin_Headers:Pin_Header_Straight_1x07, symbol Connector:Conn_01x07_Male
- added J2: Conn_01x02_Female, Terminal_Blocks:TerminalBlock_Pheonix_MKDS1.5-2pol, symbol Connector:Conn_01x02_Female
- J3: footprint Connect:BARREL_JACK -> Terminal_Blocks:TerminalBlock_Pheonix_MKDS1.5-2pol; Digikey # CP-037A-ND -> ED2561-ND
- Q1: value ZVN4206GVTA -> 2N7002E; symbol Transistor_FET:IRFS4227 -> Transistor_FET:2N7002E
Connections:
- net 12V: now also J1.7 (Pin_7), J2.2 (Pin_2)
- net GND: now also Q1.2 (S), J1.6 (Pin_6); no longer Q1.3 (S)
- net LATCH_OUT: now also Q1.3 (D), J2.1 (Pin_1); no longer Q1.2 (D)
- net READER_BUZZ: now also J1.3 (Pin_3)
- net WIEGAND_IN1: now also J1.5 (Pin_5)
- net WIEGAND_IN2: now also J1.4 (Pin_4)
- net 24_32_SWITCH: now reaches J4.4 (Pin_4)
- net 24_32_SWITCH: now also J1.1 (Pin_1)
- net READER_LED: now reaches J4.5 (Pin_5)
- net READER_LED: now also J1.2 (Pin_2)
- no-connect marks 23 -> 21
Changed lines of the file:
@@
 $EndDescr
 $Comp
-L Transistor_FET:IRFS4227 Q1
+L Transistor_FET:2N7002E Q1
 U 1 1 603A6F1F
 P 1450 5650
 F 0 "Q1" H 1654 5696 50  0000 L CNN
-F 1 "ZVN4206GVTA" H 1654 5605 50  0000 L CNN
+F 1 "2N7002E" H 1654 5605 50  0000 L CNN
 F 2 "TO_SOT_Packages_SMD:SOT-223" H 1650 5575 50  0001 L CIN
-F 3 "https://www.diodes.com/assets/Datasheets/ZVN4206GV.pdf" H 1450 5650 50  0001 L CNN
+F 3 "http://www.diodes.com/assets/Datasheets/ds30376.pdf" H 1450 5650 50  0001 L CNN
 F 4 "ZVN4206GVTR-ND" H 1450 5650 50  0001 C CNN "Digikey #"
 	1    1450 5650
@@
 Wire Wire Line
 	1100 5650 1200 5650
-Text GLabel 3650 1050 0    50   Input ~ 0
+$Comp
+L Connector:Conn_01x02_Female J2
+U 1 1 60482C20
+P 1850 3700
+F 0 "J2" H 1878 3676 50  0000 L CNN
+F 1 "Conn_01x02_Female" H 1878 3585 50  0000 L CNN
+F 2 "Terminal_Blocks:TerminalBlock_Pheonix_MKDS1.5-2pol" H 1850 3700 50  0001 C CNN
+F 3 "~" H 1850 3700 50  0001 C CNN
+F 4 "ED2561-ND" H 1850 3700 50  0001 C CNN "Digikey #"
+	1    1850 3700
+	1    0    0    -1
+$EndComp
+Text GLabel 1500 3800 0    50   Input ~ 0
 LATCH_IN
-Text GLabel 3650 1450 0    50   Input ~ 0
+Text GLabel 1500 3700 0    50   Input ~ 0
 LATCH_OUT
+Wire Wire Line
+	1500 3700 1650 3700
+Wire Wire Line
+	1650 3800 1500 3800
 Text GLabel 7800 3300 0    50   Input ~ 0
 DOOR
@@
 Text GLabel 4400 2950 0    50   Input ~ 0
 12V
+Text GLabel 5800 2950 2    50   Input ~ 0
+5V
 Wire Wire Line
 	4550 2950 4400 2950
@@
 Text GLabel 5050 5750 1    50   Input ~ 0
 WIEGAND_IN2
+Text GLabel 7750 2500 0    50   Input ~ 0
+READER_LED
 Text GLabel 7750 2600 0    50   Input ~ 0
 READER_BUZZ
-Text GLabel 3650 1750 0    50   Input ~ 0
+Text GLabel 3550 1250 0    50   Input ~ 0
 12V
-Text GLabel 3650 1350 0    50   Input ~ 0
+Text GLabel 3550 1450 0    50   Input ~ 0
 WIEGAND_IN1
-Text GLabel 3650 1150 0    50   Input ~ 0
+Text GLabel 3550 1550 0    50   Input ~ 0
 WIEGAND_IN2
-Text GLabel 3650 1250 0    50   Input ~ 0
+Text GLabel 3550 1750 0    50   Input ~ 0
+READER_LED
+Text GLabel 3550 1650 0    50   Input ~ 0
 READER_BUZZ
 $Comp
 L power:GND #PWR0109
 U 1 1 60644B08
-P 3000 1650
-F 0 "#PWR0109" H 3000 1400 50  0001 C CNN
-F 1 "GND" H 3005 1477 50  0000 C CNN
-F 2 "" H 3000 1650 50  0001 C CNN
-F 3 "" H 3000 1650 50  0001 C CNN
-	1    3000 1650
-	1    0    0    -1
-$EndComp
+P 2800 1350
+F 0 "#PWR0109" H 2800 1100 50  0001 C CNN
+F 1 "GND" H 2805 1177 50  0000 C CNN
+F 2 "" H 2800 1350 50  0001 C CNN
+F 3 "" H 2800 1350 50  0001 C CNN
+	1    2800 1350
+	1    0    0    -1
+$EndComp
+Wire Wire Line
+	3550 1250 3750 1250
+Wire Wire Line
+	3550 1450 3750 1450
+Wire Wire Line
+	3750 1550 3550 1550
+Wire Wire Line
+	3550 1650 3750 1650
 Text GLabel 1200 950  1    50   Input ~ 0
 12V
@@
 Wire Wire Line
 	1200 1100 1200 950
+Wire Wire Line
+	2800 1350 3750 1350
+$Comp
+L Connector:Conn_01x07_Male J1
+U 1 1 608355C5
+P 3950 1550
+F 0 "J1" V 3785 1528 50  0000 C CNN
+F 1 "Conn_01x07_Male" V 3876 1528 50  0000 C CNN
+F 2 "Pin_Headers:Pin_Header_Straight_1x07" H 3950 1550 50  0001 C CNN
+F 3 "~" H 3950 1550 50  0001 C CNN
+	1    3950 1550
+	-1   0    0    1
+$EndComp
+Wire Wire Line
+	3550 1750 3750 1750
+Text GLabel 3550 1850 0    50   Input ~ 0
+24_32_SWITCH
+Wire Wire Line
+	3550 1850 3750 1850
 $Comp
 L Connector:Barrel_Jack J3
@@
 F 0 "J3" H 5807 1775 50  0000 C CNN
 F 1 "Barrel_Jack" H 5807 1684 50  0000 C CNN
-F 2 "Connect:BARREL_JACK" H 5800 1410 50  0001 C CNN
-F 3 "https://www.cuidevices.com/product/resource/digikeypdf/pj-037a.pdf" H 5800 1410 50  0001 C CNN
-F 4 "CP-037A-ND" H 5750 1450 50  0001 C CNN "Digikey #"
+F 2 "Terminal_Blocks:TerminalBlock_Pheonix_MKDS1.5-2pol" H 5800 1410 50  0001 C CNN
+F 3 "~" H 5800 1410 50  0001 C CNN
+F 4 "ED2561-ND" H 5750 1450 50  0001 C CNN "Digikey #"
 	1    5750 1450
 	1    0    0    -1
@@
 Wire Wire Line
 	8900 2100 9050 2100
+Text GLabel 7750 2400 0    50   Input ~ 0
+24_32_SWITCH
 NoConn ~ 7950 3000
 NoConn ~ 7950 2900
@@
 NoConn ~ 7950 3100
 NoConn ~ 7950 3200
+Wire Wire Line
+	7750 2400 7950 2400
+Wire Wire Line
+	7750 2500 7950 2500
 Wire Wire Line
 	7750 2600 7950 2600
@@
 	1    0    0    -1
 $EndComp
-$Comp
-L Connector:DB9_Male J1
-U 1 1 61046136
-P 4050 1350
-F 0 "J1" H 4230 1396 50  0000 L CNN
-F 1 "DB9_Male" H 4230 1305 50  0000 L CNN
-F 2 "Connect:DB9FD" H 4050 1350 50  0001 C CNN
-F 3 "http://www.assmann-wsw.com/uploads/datasheets/ASS_4888_CO.pdf" H 4050 1350 50  0001 C CNN
-F 4 "AE10970-ND" H 4050 1350 50  0001 C CNN "Digikey #"
-	1    4050 1350
-	1    0    0    -1
-$EndComp
-Text GLabel 5800 2950 2    50   Input ~ 0
-5V
-Text GLabel 3650 1550 0    50   Input ~ 0
-5V
-$Comp
-L power:GND #PWR0112
-U 1 1 6104AFD6
-P 3000 950
-F 0 "#PWR0112" H 3000 700 50  0001 C CNN
-F 1 "GND" H 3005 777 50  0000 C CNN
-F 2 "" H 3000 950 50  0001 C CNN
-F 3 "" H 3000 950 50  0001 C CNN
-	1    3000 950
-	1    0    0    -1
-$EndComp
-Wire Wire Line
-	3750 950  3000 950
-Wire Wire Line
-	3650 1050 3750 1050
-Wire Wire Line
-	3750 1150 3650 1150
-Wire Wire Line
-	3650 1250 3750 1250
-Wire Wire Line
-	3750 1350 3650 1350
-Wire Wire Line
-	3650 1450 3750 1450
-Wire Wire Line
-	3750 1550 3650 1550
-Wire Wire Line
-	3000 1650 3750 1650
-Wire Wire Line
-	3750 1750 3650 1750
-NoConn ~ 7950 2400
-NoConn ~ 7950 2500
 $EndSCHEMATC
