File: esp32_pcb/esp32_doorbot.kicad_pcb (KiCad board)
At the start: 2 copper layers, 29.2 x 51.8 mm, 20 parts, among them J1 Conn_01x07_Male, J2 Conn_01x02_Female, J3 Barrel_Jack, J4 WROOM32_1, J5 WROOM32_2, Q1 ZXMP4A16G, U1 L7805

Commit message: Fixup labels
Other:
- board text added: "12/24V"
- board text added: "24/32"
- board text added: "BUZZ"
- board text added: "ESP32 Doorbot v5 By Timm Murray Copyright © 2021 BY-CC"
- board text added: "LED"
- board text added: "W1"
- board text added: "W2"
- board text removed: "ESP32 Doorbot v4 By Timm Murray Copyright © 2021 BY-CC"
